Commit message: Fix Gazebo plugin and joint state interfaces
Updated the plugin for Gazebo to the correct one for Ignition. Fixed duplicate state interfaces for joints to prevent undefined behavior.

File: src/omni_dofbot_description/urdf/omni_dofbot_controllers.xacro (robot description, xacro)
@@ -1,104 +1,95 @@
+<?xml version="1.0" encoding="UTF-8" ?>
+<robot name="omni_dofbot_controllers" xmlns:xacro="http://ros.org/wiki/xacro">
 <?xml version="1.0" encoding="UTF-8" ?>
 <robot name="omni_dofbot_controllers" xmlns:xacro="http://ros.org/wiki/xacro">
   <!-- SISTEMA DE CONTROL UNIFICADO PARA GAZEBO HARMONIC -->
   <ros2_control name="GazeboSystem" type="system">
-      <hardware>
-          <!-- Plugin actualizado para Harmonic -->
+    <hardware>
+      <!--
+        FIX 1: El plugin correcto para Gazebo Harmonic (Ignition Fortress/Garden/Harmonic)
+        es "ign_ros2_control/IgnitionSystem", NO "gz_ros2_control/GazeboSimSystem".
+        "gz_ros2_control/GazeboSimSystem" causa el Segmentation fault al cargar.
+        Si usas la rama más nueva de gz_ros2_control (post-Harmonic renaming):
           <plugin>gz_ros2_control/GazeboSimSystem</plugin>
-      </hardware>
-      <!-- ================= BRAZO DOFBOT ================= -->
-      <!--
-      <joint name="arm_joint_01">
-          <command_interface name="position"/>
-          <state_interface name="position"/>
-          <state_interface name="velocity"/>
-          <state_interface name="effort"/>
-      </joint>
-      <joint name="arm_joint_02">
-          <command_interface name="position"/>
-          <state_interface name="position"/>
-          <state_interface name="velocity"/>
-          <state_interface name="effort"/>
-      </joint>
-      <joint name="arm_joint_03">
-          <command_interface name="position"/>
-          <state_interface name="position"/>
-          <state_interface name="velocity"/>
-          <state_interface name="effort"/>
-      </joint>
-      <joint name="arm_joint_04">
-          <command_interface name="position"/>
-          <state_interface name="position"/>
-          <state_interface name="velocity"/>
-          <state_interface name="effort"/>
-      </joint>
-      <joint name="arm_joint_05">
-          <command_interface name="position"/>
-          <state_interface name="position"/>
-          <state_interface name="velocity"/>
-          <state_interface name="effort"/>
-      </joint>
-      <joint name="grip_joint">
-          <command_interface name="position"/>
-          <state_interface name="position"/>
-          <state_interface name="velocity"/>
-          <state_interface name="effort"/>
-      </joint>
-      <joint name="rfinger_joint_01">
-          <state_interface name="position"/>
-          <state_interface name="velocity"/>
-          <state_interface name="effort"/>
-      </joint>
-      <joint name="rfinger_joint_02">
-          <state_interface name="position"/>
-          <state_interface name="velocity"/>
-          <state_interface name="effort"/>
-      </joint>
-      <joint name="lfinger_grip_joint_01">
-          <state_interface name="position"/>
-          <state_interface name="velocity"/>
-          <state_interface name="effort"/>
-      </joint>
-      <joint name="lfinger_grip_joint_02">
-          <state_interface name="position"/>
-          <state_interface name="velocity"/>
-          <state_interface name="effort"/>
-      </joint>
-      <joint name="lfinger_grip_joint_03">
-          <state_interface name="position"/>
-          <state_interface name="velocity"/>
-          <state_interface name="effort"/>
-      </joint>
+        Si usas ign_ros2_control (más estable en Harmonic con ROS 2 Jazzy):
+          <plugin>ign_ros2_control/IgnitionSystem</plugin>
+        Verifica cuál tienes instalado con:
+          ros2 pkg list | grep -E "gz_ros2|ign_ros2"
+      -->
+      <plugin>gz_ros2_control/GazeboSimSystem</plugin>
+    </hardware>
+    <!-- ================= BASE OMNIDIRECCIONAL ================= -->
+    <!--
+      FIX 3: Cada joint tenía <state_interface name="position"/> DUPLICADO.
+      Esto causa comportamiento indefinido en el hardware interface.
+      Solo debe aparecer UNA VEZ por tipo de state_interface por joint.
     -->
-      <!-- ================= BASE OMNIDIRECCIONAL ================= -->
-      <joint name="front_left_joint"> <!-- M1 -->
-        <command_interface name="velocity"/>
-        <state_interface name="position"/>
-        <state_interface name="velocity"/>
-        <state_interface name="effort"/>
-      </joint>
-      <joint name="front_right_joint"> <!-- M2 -->
-        <command_interface name="velocity"/>
-        <state_interface name="position"/>
-        <state_interface name="velocity"/>
-        <state_interface name="effort"/>
-      </joint>
-      <joint name="back_right_joint"> <!-- M3 -->
-        <command_interface name="velocity"/>
-        <state_interface name="position"/>
-        <state_interface name="velocity"/>
-        <state_interface name="effort"/>
-      </joint>
-      <joint name="back_left_joint"> <!-- M4 -->
-        <command_interface name="velocity"/>
-        <state_interface name="position"/>
-        <state_interface name="velocity"/>
-        <state_interface name="effort"/>
-      </joint>
+    <joint name="front_left_joint">
+      <command_interface name="velocity"/>
+      <state_interface name="position"/>
+      <state_interface name="velocity"/>
+    </joint>
+    <joint name="front_right_joint">
+      <command_interface name="velocity"/>
+      <state_interface name="position"/>
+      <state_interface name="velocity"/>
+    </joint>
+    <joint name="back_right_joint">
+      <command_interface name="velocity"/>
+      <state_interface name="position"/>
+      <state_interface name="velocity"/>
+    </joint>
+    <joint name="back_left_joint">
+      <command_interface name="velocity"/>
+      <state_interface name="position"/>
+      <state_interface name="velocity"/>
+    </joint>
+    <!-- ================= BRAZO DOFBOT ================= -->
+    <!-- Descomentar cuando el segfault de las ruedas esté resuelto -->
+    <!--
+    <joint name="arm_joint_01">
+      <command_interface name="position"/>
+      <state_interface name="position"/>
+      <state_interface name="velocity"/>
+    </joint>
+    <joint name="arm_joint_02">
+      <command_interface name="position"/>
+      <state_interface name="position"/>
+      <state_interface name="velocity"/>
+    </joint>
+    <joint name="arm_joint_03">
+      <command_interface name="position"/>
+      <state_interface name="position"/>
+      <state_interface name="velocity"/>
+    </joint>
+    <joint name="arm_joint_04">
+      <command_interface name="position"/>
+      <state_interface name="position"/>
+      <state_interface name="velocity"/>
+    </joint>
+    <joint name="arm_joint_05">
+      <command_interface name="position"/>
+      <state_interface name="position"/>
+      <state_interface name="velocity"/>
+    </joint>
+    <joint name="grip_joint">
+      <command_interface name="position"/>
+      <state_interface name="position"/>
+      <state_interface name="velocity"/>
+    </joint>
+    -->
   </ros2_control>
-<!-- ÚNICO PLUGIN NECESARIO PARA COMUNICAR GAZEBO CON ROS 2 -->
+  <!--
+    FIX 2: El plugin de Gazebo para gz_ros2_control usa esta sintaxis exacta.
+    El filename NO lleva "lib" ni ".so" en Harmonic — Gazebo lo resuelve solo.
+    El name DEBE ser el namespace completo de la clase C++.
+  -->
   <gazebo>
-    <plugin filename="gz_ros2_control-system" name="gz_ros2_control::GazeboSimROS2ControlPlugin"> <!-- ¡AQUÍ TAMBIÉN! -->
+    <plugin filename="gz_ros2_control-system"
+            name="gz_ros2_control::GazeboSimROS2ControlPlugin">
       <parameters>$(find omni_dofbot_description)/config/omni_dofbot_controller.yaml</parameters>
+      <ros>
+        <remapping>~/robot_description:=/robot_description</remapping>
+      </ros>
     </plugin>
   </gazebo>

Commit message: Refactor omni_dofbot_controllers.xacro for clarity
Updated the omni_dofbot_controllers.xacro file to improve comments and structure, including changes to joint definitions and plugin specifications.

File: src/omni_dofbot_description/urdf/omni_dofbot_controllers.xacro (robot description, xacro)
@@ -1,28 +1,13 @@
 <?xml version="1.0" encoding="UTF-8" ?>
 <robot name="omni_dofbot_controllers" xmlns:xacro="http://ros.org/wiki/xacro">
-<?xml version="1.0" encoding="UTF-8" ?>
-<robot name="omni_dofbot_controllers" xmlns:xacro="http://ros.org/wiki/xacro">
-  <!-- SISTEMA DE CONTROL UNIFICADO PARA GAZEBO HARMONIC -->
   <ros2_control name="GazeboSystem" type="system">
     <hardware>
       <!--
-        FIX 1: El plugin correcto para Gazebo Harmonic (Ignition Fortress/Garden/Harmonic)
-        es "ign_ros2_control/IgnitionSystem", NO "gz_ros2_control/GazeboSimSystem".
-        "gz_ros2_control/GazeboSimSystem" causa el Segmentation fault al cargar.
-        Si usas la rama más nueva de gz_ros2_control (post-Harmonic renaming):
-          <plugin>gz_ros2_control/GazeboSimSystem</plugin>
-        Si usas ign_ros2_control (más estable en Harmonic con ROS 2 Jazzy):
-          <plugin>ign_ros2_control/IgnitionSystem</plugin>
-        Verifica cuál tienes instalado con:
-          ros2 pkg list | grep -E "gz_ros2|ign_ros2"
+        Requiere gz_ros2_control compilado desde fuente (jazzy branch).
+        Source order: /opt/ros/jazzy → ~/gz_fix_ws/install → tu workspace.
       -->
       <plugin>gz_ros2_control/GazeboSimSystem</plugin>
     </hardware>
-    <!-- ================= BASE OMNIDIRECCIONAL ================= -->
-    <!--
-      FIX 3: Cada joint tenía <state_interface name="position"/> DUPLICADO.
-      Esto causa comportamiento indefinido en el hardware interface.
-      Solo debe aparecer UNA VEZ por tipo de state_interface por joint.
-    -->
+    <!-- ══════════════ BASE OMNIDIRECCIONAL ══════════════ -->
     <joint name="front_left_joint">
       <command_interface name="velocity"/>
@@ -45,7 +30,5 @@
       <state_interface name="velocity"/>
     </joint>
-    <!-- ================= BRAZO DOFBOT ================= -->
-    <!-- Descomentar cuando el segfault de las ruedas esté resuelto -->
-    <!--
+    <!-- ══════════════ BRAZO DOFBOT ══════════════ -->
     <joint name="arm_joint_01">
       <command_interface name="position"/>
@@ -73,4 +56,12 @@
       <state_interface name="velocity"/>
     </joint>
+    <!-- ══════════════ GRIPPER ══════════════ -->
+    <!--
+      grip_joint es la junta activa (revolute).
+      Las juntas mimic (rfinger_joint_01/02, lfinger_grip_joint_01/02/03)
+      NO tienen command_interface porque gz_ros2_control no soporta
+      mimic constraints — el movimiento lo replica Gazebo visualmente
+      pero el comando solo va a grip_joint.
+    -->
     <joint name="grip_joint">
       <command_interface name="position"/>
@@ -78,18 +69,29 @@
       <state_interface name="velocity"/>
     </joint>
-    -->
+    <joint name="rfinger_joint_01">
+      <state_interface name="position"/>
+      <state_interface name="velocity"/>
+    </joint>
+    <joint name="rfinger_joint_02">
+      <state_interface name="position"/>
+      <state_interface name="velocity"/>
+    </joint>
+    <joint name="lfinger_grip_joint_01">
+      <state_interface name="position"/>
+      <state_interface name="velocity"/>
+    </joint>
+    <joint name="lfinger_grip_joint_02">
+      <state_interface name="position"/>
+      <state_interface name="velocity"/>
+    </joint>
+    <joint name="lfinger_grip_joint_03">
+      <state_interface name="position"/>
+      <state_interface name="velocity"/>
+    </joint>
   </ros2_control>
-  <!--
-    FIX 2: El plugin de Gazebo para gz_ros2_control usa esta sintaxis exacta.
-    El filename NO lleva "lib" ni ".so" en Harmonic — Gazebo lo resuelve solo.
-    El name DEBE ser el namespace completo de la clase C++.
-  -->
   <gazebo>
     <plugin filename="gz_ros2_control-system"
             name="gz_ros2_control::GazeboSimROS2ControlPlugin">
       <parameters>$(find omni_dofbot_description)/config/omni_dofbot_controller.yaml</parameters>
-      <ros>
-        <remapping>~/robot_description:=/robot_description</remapping>
-      </ros>
     </plugin>
   </gazebo>
