Commit message: Creación de mapa y uso de ROS2 navegation para sintonizar PID basado en trayectoria

File: install/omni_dofbot_description/share/omni_dofbot_description/urdf/omni_dofbot_controllers.xacro (robot description, xacro)
@@ -1,103 +1,97 @@
 <?xml version="1.0" encoding="UTF-8" ?>
 <robot name="omni_dofbot_controllers" xmlns:xacro="http://ros.org/wiki/xacro">
-  <!-- SISTEMA DE CONTROL UNIFICADO PARA GAZEBO HARMONIC -->
-  <ros2_control name="GazeboSystem" type="system">
-      <hardware>
-          <!-- Plugin actualizado para Harmonic -->
-          <plugin>gz_ros2_control/GazeboSimSystem</plugin>
-      </hardware>
-      <!-- ================= BRAZO DOFBOT ================= -->
-      <!--
-      <joint name="arm_joint_01">
-          <command_interface name="position"/>
-          <state_interface name="position"/>
-          <state_interface name="velocity"/>
-          <state_interface name="effort"/>
-      </joint>
-      <joint name="arm_joint_02">
-          <command_interface name="position"/>
-          <state_interface name="position"/>
-          <state_interface name="velocity"/>
-          <state_interface name="effort"/>
-      </joint>
-      <joint name="arm_joint_03">
-          <command_interface name="position"/>
-          <state_interface name="position"/>
-          <state_interface name="velocity"/>
-          <state_interface name="effort"/>
-      </joint>
-      <joint name="arm_joint_04">
-          <command_interface name="position"/>
-          <state_interface name="position"/>
-          <state_interface name="velocity"/>
-          <state_interface name="effort"/>
-      </joint>
-      <joint name="arm_joint_05">
-          <command_interface name="position"/>
-          <state_interface name="position"/>
-          <state_interface name="velocity"/>
-          <state_interface name="effort"/>
-      </joint>
-      <joint name="grip_joint">
-          <command_interface name="position"/>
-          <state_interface name="position"/>
-          <state_interface name="velocity"/>
-          <state_interface name="effort"/>
-      </joint>
-      <joint name="rfinger_joint_01">
-          <state_interface name="position"/>
-          <state_interface name="velocity"/>
-          <state_interface name="effort"/>
-      </joint>
-      <joint name="rfinger_joint_02">
-          <state_interface name="position"/>
-          <state_interface name="velocity"/>
-          <state_interface name="effort"/>
-      </joint>
-      <joint name="lfinger_grip_joint_01">
-          <state_interface name="position"/>
-          <state_interface name="velocity"/>
-          <state_interface name="effort"/>
-      </joint>
-      <joint name="lfinger_grip_joint_02">
-          <state_interface name="position"/>
-          <state_interface name="velocity"/>
-          <state_interface name="effort"/>
-      </joint>
-      <joint name="lfinger_grip_joint_03">
-          <state_interface name="position"/>
-          <state_interface name="velocity"/>
-          <state_interface name="effort"/>
-      </joint>
-    -->
-      <!-- ================= BASE OMNIDIRECCIONAL ================= -->
-      <joint name="front_left_joint"> <!-- M1 -->
-        <command_interface name="velocity"/>
-        <state_interface name="position"/>
-        <state_interface name="velocity"/>
-        <state_interface name="effort"/>
-      </joint>
-      <joint name="front_right_joint"> <!-- M2 -->
-        <command_interface name="velocity"/>
-        <state_interface name="position"/>
-        <state_interface name="velocity"/>
-        <state_interface name="effort"/>
-      </joint>
-      <joint name="back_right_joint"> <!-- M3 -->
-        <command_interface name="velocity"/>
-        <state_interface name="position"/>
-        <state_interface name="velocity"/>
-        <state_interface name="effort"/>
-      </joint>
-      <joint name="back_left_joint"> <!-- M4 -->
-        <command_interface name="velocity"/>
-        <state_interface name="position"/>
-        <state_interface name="velocity"/>
-        <state_interface name="effort"/>
-      </joint>
+  <!--
+    NOMBRE ÚNICO: "OmniDofbotSystem" para evitar conflicto con el bloque
+    name="GazeboSystem" que viene de dofbot_arm_urdf.xacro →
+    trajectory_controller.xacro (Gazebo Classic).
+    gz_ros2_control 1.2.x registra AMBOS bloques cuando tienen nombres
+    distintos, pero solo activa el hardware del bloque cuyo plugin
+    (GazeboSimSystem) matchea el motor de simulación actual.
+    El bloque "GazeboSystem" con plugin gazebo_ros2_control/GazeboSystem
+    (Gazebo Classic) falla silenciosamente y se ignora en Harmonic.
+    El bloque "OmniDofbotSystem" con gz_ros2_control/GazeboSimSystem
+    se activa correctamente y registra TODOS los joints aquí declarados.
+  -->
+  <ros2_control name="OmniDofbotSystem" type="system">
+    <hardware>
+      <plugin>gz_ros2_control/GazeboSimSystem</plugin>
+    </hardware>
+    <!-- ══════════════ BASE OMNIDIRECCIONAL ══════════════ -->
+    <joint name="front_left_joint">
+      <command_interface name="velocity"/>
+      <state_interface name="position"/>
+      <state_interface name="velocity"/>
+    </joint>
+    <joint name="front_right_joint">
+      <command_interface name="velocity"/>
+      <state_interface name="position"/>
+      <state_interface name="velocity"/>
+    </joint>
+    <joint name="back_right_joint">
+      <command_interface name="velocity"/>
+      <state_interface name="position"/>
+      <state_interface name="velocity"/>
+    </joint>
+    <joint name="back_left_joint">
+      <command_interface name="velocity"/>
+      <state_interface name="position"/>
+      <state_interface name="velocity"/>
+    </joint>
+    <!-- ══════════════ BRAZO DOFBOT ══════════════ -->
+    <joint name="arm_joint_01">
+      <command_interface name="position"/>
+      <state_interface name="position"/>
+      <state_interface name="velocity"/>
+    </joint>
+    <joint name="arm_joint_02">
+      <command_interface name="position"/>
+      <state_interface name="position"/>
+      <state_interface name="velocity"/>
+    </joint>
+    <joint name="arm_joint_03">
+      <command_interface name="position"/>
+      <state_interface name="position"/>
+      <state_interface name="velocity"/>
+    </joint>
+    <joint name="arm_joint_04">
+      <command_interface name="position"/>
+      <state_interface name="position"/>
+      <state_interface name="velocity"/>
+    </joint>
+    <joint name="arm_joint_05">
+      <command_interface name="position"/>
+      <state_interface name="position"/>
+      <state_interface name="velocity"/>
+    </joint>
+    <!-- ══════════════ GRIPPER ══════════════ -->
+    <joint name="grip_joint">
+      <command_interface name="position"/>
+      <state_interface name="position"/>
+      <state_interface name="velocity"/>
+    </joint>
+    <joint name="rfinger_joint_01">
+      <state_interface name="position"/>
+      <state_interface name="velocity"/>
+    </joint>
+    <joint name="rfinger_joint_02">
+      <state_interface name="position"/>
+      <state_interface name="velocity"/>
+    </joint>
+    <joint name="lfinger_grip_joint_01">
+      <state_interface name="position"/>
+      <state_interface name="velocity"/>
+    </joint>
+    <joint name="lfinger_grip_joint_02">
+      <state_interface name="position"/>
+      <state_interface name="velocity"/>
+    </joint>
+    <joint name="lfinger_grip_joint_03">
+      <state_interface name="position"/>
+      <state_interface name="velocity"/>
+    </joint>
   </ros2_control>
-<!-- ÚNICO PLUGIN NECESARIO PARA COMUNICAR GAZEBO CON ROS 2 -->
   <gazebo>
-    <plugin filename="gz_ros2_control-system" name="gz_ros2_control::GazeboSimROS2ControlPlugin"> <!-- ¡AQUÍ TAMBIÉN! -->
+    <plugin filename="gz_ros2_control-system"
+            name="gz_ros2_control::GazeboSimROS2ControlPlugin">
       <parameters>$(find omni_dofbot_description)/config/omni_dofbot_controller.yaml</parameters>
     </plugin>
