Commit message: Cambios en las pruebas para sintonización debido a la limitación de movimiento en Y para las ruedas del robot, correción de parametros de velocidad en las ruedas para permitir al robot alcanzar la velocidad máxima

File: install/omni_description/share/omni_description/urdf/omni_urdf.xacro (robot description, xacro)
@@ -39,20 +39,15 @@
             <origin xyz="1.9051E-06 -2.3183E-07 -0.00064079" rpy="0 0 0"/>
             <mass value="0.051532"/>
-            <inertia ixx="1.4595E-05" ixy="-4.3975E-10" ixz="4.415E-10"
-                     iyy="1.4594E-05" iyz="-1.7476E-09" izz="2.4264E-05"/>
+            <inertia ixx="1.4595E-05" ixy="-4.3975E-10" ixz="4.415E-10" iyy="1.4594E-05" iyz="-1.7476E-09" izz="2.4264E-05"/>
         </inertial>
         <visual>
             <origin xyz="0 0 0" rpy="0 0 0"/>
-            <geometry>
-                <mesh filename="${f_r_wheel}"/>
-            </geometry>
-            <material name="">
-                <color rgba="0.7 0.7 0.7 1"/>
-            </material>
+            <geometry><mesh filename="${f_r_wheel}"/></geometry>
+            <material name=""><color rgba="0.7 0.7 0.7 1"/></material>
         </visual>
         <collision>
             <origin xyz="0 0 0" rpy="0 0 0"/>
             <geometry>
-                <mesh filename="${f_r_wheel}"/>
+                <sphere radius="0.04"/>
             </geometry>
         </collision>
@@ -63,5 +58,5 @@
         <child link="front_right_wheel"/>
         <axis xyz="0 0 1" rpy="0 0 0"/>
-        <limit effort="100" velocity="1"/>
+        <limit effort="100" velocity="17.5"/>
     </joint>
     <link name="front_left_wheel">
@@ -69,20 +64,15 @@
             <origin xyz="2.3728E-06 -9.4228E-07 0.00064068" rpy="0 0 0"/>
             <mass value="0.051543"/>
-            <inertia ixx="1.4597E-05" ixy="-4.7945E-10" ixz="-2.4786E-10"
-                     iyy="1.4598E-05" iyz="1.7972E-09" izz="2.4267E-05"/>
+            <inertia ixx="1.4597E-05" ixy="-4.7945E-10" ixz="-2.4786E-10" iyy="1.4598E-05" iyz="1.7972E-09" izz="2.4267E-05"/>
         </inertial>
         <visual>
             <origin xyz="0 0 0" rpy="0 0 0"/>
-            <geometry>
-                <mesh filename="${f_l_wheel}"/>
-            </geometry>
-            <material name="">
-                <color rgba="0.7 0.7 0.7 1"/>
-            </material>
+            <geometry><mesh filename="${f_l_wheel}"/></geometry>
+            <material name=""><color rgba="0.7 0.7 0.7 1"/></material>
         </visual>
         <collision>
             <origin xyz="0 0 0" rpy="0 0 0"/>
             <geometry>
-                <mesh filename="${f_l_wheel}"/>
+                <sphere radius="0.04"/>
             </geometry>
         </collision>
@@ -93,5 +83,5 @@
         <child link="front_left_wheel"/>
         <axis xyz="0 0 1" rpy="0 0 0"/>
-        <limit effort="100" velocity="1"/>
+        <limit effort="100" velocity="17.5"/>
     </joint>
     <link name="back_right_wheel">
@@ -99,20 +89,15 @@
             <origin xyz="-1.75924169923403E-06 1.28388821071107E-06 -0.000590549296238266" rpy="0 0 0"/>
             <mass value="0.051540174053366"/>
-            <inertia ixx="1.45974152250002E-05" ixy="1.94850559178397E-10" ixz="-1.61846387282284E-09"
-                     iyy="1.4596501955693E-05" iyz="-6.27904057423818E-10" izz="2.42663091380451E-05"/>
+            <inertia ixx="1.45974152250002E-05" ixy="1.94850559178397E-10" ixz="-1.61846387282284E-09" iyy="1.4596501955693E-05" iyz="-6.27904057423818E-10" izz="2.42663091380451E-05"/>
         </inertial>
         <visual>
             <origin xyz="0 0 0" rpy="0 0 0"/>
-            <geometry>
-                <mesh filename="${b_r_wheel}"/>
-            </geometry>
-            <material name="">
-                <color rgba="0.7 0.7 0.7 1"/>
-            </material>
+            <geometry><mesh filename="${b_r_wheel}"/></geometry>
+            <material name=""><color rgba="0.7 0.7 0.7 1"/></material>
         </visual>
         <collision>
             <origin xyz="0 0 0" rpy="0 0 0"/>
             <geometry>
-                <mesh filename="${b_r_wheel}"/>
+                <sphere radius="0.04"/>
             </geometry>
         </collision>
@@ -123,5 +108,5 @@
         <child link="back_right_wheel"/>
         <axis xyz="0 0 1" rpy="0 0 0"/>
-        <limit effort="100" velocity="1"/>
+        <limit effort="100" velocity="17.5"/>
     </joint>
     <link name="back_left_wheel">
@@ -129,20 +114,15 @@
             <origin xyz="-4.01213085227115E-07 2.04910264598596E-06 0.000590775697051377" rpy="0 0 0"/>
             <mass value="0.0515309299357028"/>
-            <inertia ixx="1.45942986129926E-05" ixy="-3.19787215398093E-10" ixz="1.74943062058915E-09"
-                     iyy="1.45948727598913E-05" iyz="1.61769812110049E-10" izz="2.4263683888153E-05"/>
+            <inertia ixx="1.45942986129926E-05" ixy="-3.19787215398093E-10" ixz="1.74943062058915E-09" iyy="1.45948727598913E-05" iyz="1.61769812110049E-10" izz="2.4263683888153E-05"/>
         </inertial>
         <visual>
             <origin xyz="0 0 0" rpy="0 0 0"/>
-            <geometry>
-                <mesh filename="${b_l_wheel}"/>
-            </geometry>
-            <material name="">
-                <color rgba="0.7 0.7 0.7 1"/>
-            </material>
+            <geometry><mesh filename="${b_l_wheel}"/></geometry>
+            <material name=""><color rgba="0.7 0.7 0.7 1"/></material>
         </visual>
         <collision>
             <origin xyz="0 0 0" rpy="0 0 0"/>
             <geometry>
-                <mesh filename="${b_l_wheel}"/>
+                <sphere radius="0.04"/>
             </geometry>
         </collision>
@@ -153,5 +133,25 @@
         <child link="back_left_wheel"/>
         <axis xyz="0 0 1" rpy="0 0 0"/>
-        <limit effort="100" velocity="1"/>
+        <limit effort="100" velocity="17.5"/>
     </joint>
+    <gazebo reference="front_left_wheel">
+        <mu1>1.0</mu1>
+        <mu2>0.0</mu2>
+        <fdir1>1 -1 0</fdir1>
+    </gazebo>
+    <gazebo reference="front_right_wheel">
+        <mu1>1.0</mu1>
+        <mu2>0.0</mu2>
+        <fdir1>1 1 0</fdir1>
+    </gazebo>
+    <gazebo reference="back_left_wheel">
+        <mu1>1.0</mu1>
+        <mu2>0.0</mu2>
+        <fdir1>1 1 0</fdir1>
+    </gazebo>
+    <gazebo reference="back_right_wheel">
+        <mu1>1.0</mu1>
+        <mu2>0.0</mu2>
+        <fdir1>1 -1 0</fdir1>
+    </gazebo>
 </robot>

Commit message: Corrección en archivo Xacro manteniendo el mesh de la llanta

File: install/omni_description/share/omni_description/urdf/omni_urdf.xacro (robot description, xacro)
@@ -39,15 +39,20 @@
             <origin xyz="1.9051E-06 -2.3183E-07 -0.00064079" rpy="0 0 0"/>
             <mass value="0.051532"/>
-            <inertia ixx="1.4595E-05" ixy="-4.3975E-10" ixz="4.415E-10" iyy="1.4594E-05" iyz="-1.7476E-09" izz="2.4264E-05"/>
+            <inertia ixx="1.4595E-05" ixy="-4.3975E-10" ixz="4.415E-10"
+                     iyy="1.4594E-05" iyz="-1.7476E-09" izz="2.4264E-05"/>
         </inertial>
         <visual>
             <origin xyz="0 0 0" rpy="0 0 0"/>
-            <geometry><mesh filename="${f_r_wheel}"/></geometry>
-            <material name=""><color rgba="0.7 0.7 0.7 1"/></material>
+            <geometry>
+                <mesh filename="${f_r_wheel}"/>
+            </geometry>
+            <material name="">
+                <color rgba="0.7 0.7 0.7 1"/>
+            </material>
         </visual>
         <collision>
             <origin xyz="0 0 0" rpy="0 0 0"/>
             <geometry>
-                <sphere radius="0.04"/>
+                <mesh filename="${f_r_wheel}"/>
             </geometry>
         </collision>
@@ -64,15 +69,20 @@
             <origin xyz="2.3728E-06 -9.4228E-07 0.00064068" rpy="0 0 0"/>
             <mass value="0.051543"/>
-            <inertia ixx="1.4597E-05" ixy="-4.7945E-10" ixz="-2.4786E-10" iyy="1.4598E-05" iyz="1.7972E-09" izz="2.4267E-05"/>
+            <inertia ixx="1.4597E-05" ixy="-4.7945E-10" ixz="-2.4786E-10"
+                     iyy="1.4598E-05" iyz="1.7972E-09" izz="2.4267E-05"/>
         </inertial>
         <visual>
             <origin xyz="0 0 0" rpy="0 0 0"/>
-            <geometry><mesh filename="${f_l_wheel}"/></geometry>
-            <material name=""><color rgba="0.7 0.7 0.7 1"/></material>
+            <geometry>
+                <mesh filename="${f_l_wheel}"/>
+            </geometry>
+            <material name="">
+                <color rgba="0.7 0.7 0.7 1"/>
+            </material>
         </visual>
         <collision>
             <origin xyz="0 0 0" rpy="0 0 0"/>
             <geometry>
-                <sphere radius="0.04"/>
+                <mesh filename="${f_l_wheel}"/>
             </geometry>
         </collision>
@@ -89,15 +99,20 @@
             <origin xyz="-1.75924169923403E-06 1.28388821071107E-06 -0.000590549296238266" rpy="0 0 0"/>
             <mass value="0.051540174053366"/>
-            <inertia ixx="1.45974152250002E-05" ixy="1.94850559178397E-10" ixz="-1.61846387282284E-09" iyy="1.4596501955693E-05" iyz="-6.27904057423818E-10" izz="2.42663091380451E-05"/>
+            <inertia ixx="1.45974152250002E-05" ixy="1.94850559178397E-10" ixz="-1.61846387282284E-09"
+                     iyy="1.4596501955693E-05" iyz="-6.27904057423818E-10" izz="2.42663091380451E-05"/>
         </inertial>
         <visual>
             <origin xyz="0 0 0" rpy="0 0 0"/>
-            <geometry><mesh filename="${b_r_wheel}"/></geometry>
-            <material name=""><color rgba="0.7 0.7 0.7 1"/></material>
+            <geometry>
+                <mesh filename="${b_r_wheel}"/>
+            </geometry>
+            <material name="">
+                <color rgba="0.7 0.7 0.7 1"/>
+            </material>
         </visual>
         <collision>
             <origin xyz="0 0 0" rpy="0 0 0"/>
             <geometry>
-                <sphere radius="0.04"/>
+                <mesh filename="${b_r_wheel}"/>
             </geometry>
         </collision>
@@ -114,15 +129,20 @@
             <origin xyz="-4.01213085227115E-07 2.04910264598596E-06 0.000590775697051377" rpy="0 0 0"/>
             <mass value="0.0515309299357028"/>
-            <inertia ixx="1.45942986129926E-05" ixy="-3.19787215398093E-10" ixz="1.74943062058915E-09" iyy="1.45948727598913E-05" iyz="1.61769812110049E-10" izz="2.4263683888153E-05"/>
+            <inertia ixx="1.45942986129926E-05" ixy="-3.19787215398093E-10" ixz="1.74943062058915E-09"
+                     iyy="1.45948727598913E-05" iyz="1.61769812110049E-10" izz="2.4263683888153E-05"/>
         </inertial>
         <visual>
             <origin xyz="0 0 0" rpy="0 0 0"/>
-            <geometry><mesh filename="${b_l_wheel}"/></geometry>
-            <material name=""><color rgba="0.7 0.7 0.7 1"/></material>
+            <geometry>
+                <mesh filename="${b_l_wheel}"/>
+            </geometry>
+            <material name="">
+                <color rgba="0.7 0.7 0.7 1"/>
+            </material>
         </visual>
         <collision>
             <origin xyz="0 0 0" rpy="0 0 0"/>
             <geometry>
-                <sphere radius="0.04"/>
+                <mesh filename="${b_l_wheel}"/>
             </geometry>
         </collision>
@@ -135,23 +155,3 @@
         <limit effort="100" velocity="17.5"/>
     </joint>
-    <gazebo reference="front_left_wheel">
-        <mu1>1.0</mu1>
-        <mu2>0.0</mu2>
-        <fdir1>1 -1 0</fdir1>
-    </gazebo>
-    <gazebo reference="front_right_wheel">
-        <mu1>1.0</mu1>
-        <mu2>0.0</mu2>
-        <fdir1>1 1 0</fdir1>
-    </gazebo>
-    <gazebo reference="back_left_wheel">
-        <mu1>1.0</mu1>
-        <mu2>0.0</mu2>
-        <fdir1>1 1 0</fdir1>
-    </gazebo>
-    <gazebo reference="back_right_wheel">
-        <mu1>1.0</mu1>
-        <mu2>0.0</mu2>
-        <fdir1>1 -1 0</fdir1>
-    </gazebo>
 </robot>
