Commit message: Inclusión de un ZN en lazo abierto

File: install/dofbot_description/share/dofbot_description/urdf/dofbot_arm_urdf.xacro (robot description, xacro)
@@ -165,4 +165,22 @@
         <limit lower="-1.5708" upper="3.14159" effort="100" velocity="1" />
     </joint>
+    <link name="payload_link">
+        <inertial>
+            <origin xyz="0 0 0.02" rpy="0 0 0" />
+            <mass value="1.0" />
+            <inertia ixx="0.001" ixy="0.0" ixz="0.0" iyy="0.001" iyz="0.0" izz="0.001" />
+        </inertial>
+        <visual>
+            <origin xyz="0 0 0.02" rpy="0 0 0" />
+            <geometry>
+                <sphere radius="0.025"/> </geometry>
+            <material name="eerie_black" />
+        </visual>
+    </link>
+    <joint name="payload_fixed_joint" type="fixed">
+        <origin xyz="0 0 0" rpy="0 0 0" />
+        <parent link="arm_link_05" />
+        <child link="payload_link" />
+    </joint>
     <!-- Dofbot Arm Gripper Assembly-->
     <!-- Dofbot Arm Gripper Right Grip finger link 01 -->

Commit message: Corrección de error en teleport por volcadura

File: install/dofbot_description/share/dofbot_description/urdf/dofbot_arm_urdf.xacro (robot description, xacro)
@@ -165,12 +165,14 @@
         <limit lower="-1.5708" upper="3.14159" effort="100" velocity="1" />
     </joint>
+    <xacro:arg name="payload_mass_val" default="0.150" />
+    <xacro:property name="payload_mass_val" value="$(arg payload_mass_val)" />
     <link name="payload_link">
         <inertial>
-            <origin xyz="0 0 0.02" rpy="0 0 0" />
-            <mass value="1.0" />
+            <origin xyz="0 0 0.005" rpy="0 0 0" />
+            <mass value="${payload_mass_val}" />
             <inertia ixx="0.001" ixy="0.0" ixz="0.0" iyy="0.001" iyz="0.0" izz="0.001" />
         </inertial>
         <visual>
-            <origin xyz="0 0 0.02" rpy="0 0 0" />
+            <origin xyz="0 0 0.005" rpy="0 0 0" />
             <geometry>
                 <sphere radius="0.025"/> </geometry>
