Commit message: Versión final

File: src/dofbot_description/urdf/dofbot_arm_urdf.xacro (robot description, xacro)
@@ -165,24 +165,4 @@
         <limit lower="-1.5708" upper="3.14159" effort="100" velocity="1" />
     </joint>
-    <xacro:arg name="payload_mass_val" default="0.0" />
-    <xacro:property name="payload_mass_val" value="$(arg payload_mass_val)" />
-    <link name="payload_link">
-        <inertial>
-            <origin xyz="0 0 0.005" rpy="0 0 0" />
-            <mass value="${payload_mass_val}" />
-            <inertia ixx="0.001" ixy="0.0" ixz="0.0" iyy="0.001" iyz="0.0" izz="0.001" />
-        </inertial>
-        <visual>
-            <origin xyz="0 0 0.005" rpy="0 0 0" />
-            <geometry>
-                <sphere radius="0.025"/> </geometry>
-            <material name="eerie_black" />
-        </visual>
-    </link>
-    <joint name="payload_fixed_joint" type="fixed">
-        <origin xyz="0 0 0" rpy="0 0 0" />
-        <parent link="arm_link_05" />
-        <child link="payload_link" />
-    </joint>
     <!-- Dofbot Arm Gripper Assembly-->
     <!-- Dofbot Arm Gripper Right Grip finger link 01 -->

File: src/omni_description/urdf/omni_urdf.xacro (robot description, xacro)
@@ -63,5 +63,5 @@
         <child link="front_right_wheel"/>
         <axis xyz="0 0 1" rpy="0 0 0"/>
-        <limit effort="100" velocity="17.5"/>
+        <limit effort="100" velocity="25.0"/>
     </joint>
     <link name="front_left_wheel">
@@ -93,5 +93,5 @@
         <child link="front_left_wheel"/>
         <axis xyz="0 0 1" rpy="0 0 0"/>
-        <limit effort="100" velocity="17.5"/>
+        <limit effort="100" velocity="25.0"/>
     </joint>
     <link name="back_right_wheel">
@@ -123,5 +123,5 @@
         <child link="back_right_wheel"/>
         <axis xyz="0 0 1" rpy="0 0 0"/>
-        <limit effort="100" velocity="17.5"/>
+        <limit effort="100" velocity="25.0"/>
     </joint>
     <link name="back_left_wheel">
@@ -153,5 +153,5 @@
         <child link="back_left_wheel"/>
         <axis xyz="0 0 1" rpy="0 0 0"/>
-        <limit effort="100" velocity="17.5"/>
+        <limit effort="100" velocity="25.0"/>
     </joint>
 </robot>
